File: KiCad/Parallel_to_ESP32.kicad_pcb (KiCad board)
At the start: 2 copper layers, 47 x 50 mm, 28 parts, among them J1 DB25_Male, J2 Micro_SD_Card_Socket, J3 Conn_02x02_Top_Bottom, J4 Conn_02x02_Top_Bottom, U1 ESP32-DEVKIT-V1, U2 SN74CB3T16210

Commit message: Added OSHW-silkscreen logos
Parts:
- added REF**: OSHW-Logo2_14.6x12mm_SilkScreen, Symbol:OSHW-Logo2_14.6x12mm_SilkScreen, B.Cu at (148.2, 113.5)
- added REF**: OSHW-Symbol_6.7x6mm_SilkScreen, Symbol:OSHW-Symbol_6.7x6mm_SilkScreen, F.Cu at (165.6, 98.3)
